Commit message: modify : scale up 1 -> 2

File: gym_pybullet_drones/assets/cf2x.urdf (robot description, URDF)
Before this commit: robot cf2, 6 links, 5 joints
Links:
- link base_link: geometry collision cylinder length=.025 radius=.06; visual mesh filename=./cf2.dae scale=2 2 2

Commit message: fix: 드론 바퀴 단걸로 변경

File: gym_pybullet_drones/assets/cf2x.urdf (robot description, URDF)
Before this commit: robot cf2, 6 links, 5 joints
Links:
- added link wheel_back_left_link, mass 0.0001; collision cylinder length=0.02 radius=0.015; visual cylinder length=0.02 radius=0.015
- added link wheel_back_right_link, mass 0.0001; collision cylinder length=0.02 radius=0.015; visual cylinder length=0.02 radius=0.015
- added link wheel_front_left_link, mass 0.0001; collision cylinder length=0.02 radius=0.015; visual cylinder length=0.02 radius=0.015
- added link wheel_front_right_link, mass 0.0001; collision cylinder length=0.02 radius=0.015; visual cylinder length=0.02 radius=0.015
Joints:
- added joint wheel_back_left_joint: type continuous, parent base_link, child wheel_back_left_link, origin xyz=-0.03 0.03 -0.02 rpy=-1.5708 0 0, axis 0 0 1
- added joint wheel_back_right_joint: type continuous, parent base_link, child wheel_back_right_link, origin xyz=-0.03 -0.03 -0.02 rpy=-1.5708 0 0, axis 0 0 1
- added joint wheel_front_left_joint: type continuous, parent base_link, child wheel_front_left_link, origin xyz=0.03 0.03 -0.02 rpy=-1.5708 0 0, axis 0 0 1
- added joint wheel_front_right_joint: type continuous, parent base_link, child wheel_front_right_link, origin xyz=0.03 -0.03 -0.02 rpy=-1.5708 0 0, axis 0 0 1

Commit message: fix: pid.py로부터 구현

File: gym_pybullet_drones/assets/cf2x.urdf (robot description, URDF)
Before this commit: robot cf2, 10 links, 9 joints
Links:
- link wheel_back_left_link: mass 0.0001 -> 0
- link wheel_back_right_link: mass 0.0001 -> 0
- link wheel_front_left_link: mass 0.0001 -> 0
- link wheel_front_right_link: mass 0.0001 -> 0
